File: KICAD Projects/Primis_Versipellis/Primis_Versipellis.kicad_pcb (KiCad board)
At the start: 2 copper layers, 50 x 26 mm, 28 parts, among them J2 USB_A, J3 Conn_01x05_Pin, U1 nRF52833_QDxx, Y1 32MHz

Commit message: Versipellis Update 1
-Fixed VDD
Routing:
- net VDD_nRF: track 34.0 -> 93.4 mm, vias 0 -> 4
- net GND: track 36.5 -> 39.1 mm
