File: KICAD Projects/Primis_Versipellis/Primis_Versipellis.kicad_sch (KiCad schematic)
At the start: 27 parts, among them J2 USB_A, J3 Conn_01x05_Pin, U1 nRF52833_QDxx, Y1 32MHz

Commit message: Versipellis Update 1
-Fixed VDD
Other:
- moved on the sheet: C1, C10, C11, C2, C29, C3, C30, C31, C4, C5, C6, C7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
